File: V4LPH4.kicad_pcb (KiCad board)
At the start: 2 copper layers, 242.9 x 96.6 mm, 132 parts, among them SW1 SW_PUSH, SW2 SW_PUSH, U1 SRV05-4, U2 ATmega32U4-M, X1 Crystal_GND24_Small

Commit message: route
Parts:
- K_SPACE41, K_SPACE46: footprint MX_Only:MXOnly-1U-NoLED -> MX_Only:MXOnly-1.25U-NoLED
- K_SPACE42, K_SPACE45: footprint MX_Only:MXOnly-1.25U-NoLED -> MX_Only:MXOnly-1U-NoLED
- K_SPACE43: footprint MX_Only:MXOnly-1.75U-NoLED -> MX_Only:MXOnly-1.5U-NoLED
- K_SPACE44: footprint MX_Only:MXOnly-1.5U-NoLED -> MX_Only:MXOnly-1.75U-NoLED
- moved R1 10.1 mm to (85.7, 61.1), turned to 180 degrees
- moved SW1 9.52 mm to (83.3, 56.8), turned to 180 degrees
- moved SW2 9.52 mm to (83.3, 56.8), turned to 0 degrees
- moved R4 8.99 mm to (34.9, 46.6)
- moved D2 6.70 mm to (31.5, 46.6), turned to 180 degrees
- moved D3 5.89 mm to (31.5, 52.1), turned to 180 degrees
- moved F1 4.27 mm to (61.9, 57.9), turned to -45 degrees
- moved R3 2.83 mm to (34.9, 41.1)
- moved D1 2.65 mm to (31.5, 41.1), turned to 180 degrees
- moved D_SPACE46 2.39 mm to (212.6, 124.3)
- moved D_SPACE42 2.39 mm to (110.3, 124.3)
- moved D_SPACE41 2.39 mm to (88.8, 124.3)
- moved D_SPACE45 2.38 mm to (191.2, 124.3)
- moved K_SPACE41 2.38 mm to (85.7, 123.5)
- moved K_SPACE42 2.38 mm to (107.2, 123.5)
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Connections:
- K_SPACE33 pad 1: col11 -> col12
- K_SPACE44 pad 1: col7 -> col8
- K_SPACE45 pad 1: col8 -> col9
- K_SPACE46 pad 1: col9 -> col10
- K_SPACE47 pad 1: col10 -> col11
- U2 pad 10: unconnected-(U2-Pad10) -> LED_2
- U2 pad 11: unconnected-(U2-Pad11) -> LED_3
- U2 pad 12: row0 -> row4
- U2 pad 20: PD2 -> row0
- U2 pad 22: PD5 -> unconnected-(U2-Pad22)
- U2 pad 30: row2 -> row1
- U2 pad 31: row3 -> row2
- U2 pad 32: unconnected-(U2-Pad32) -> row3
- U2 pad 36: row4 -> unconnected-(U2-Pad36)
- U2 pad 37: row1 -> col5
- U2 pad 8: col5 -> unconnected-(U2-Pad8)
- U2 pad 9: unconnected-(U2-Pad9) -> LED_1
Routing:
- net GND: track 908.9 -> 55.1 mm, vias 38 -> 22
- net row2: track 534.3 -> 249.8 mm, vias 3 -> 0
- net row3: track 4.93 -> 274.0 mm, vias 0 -> 2
- net row1: track 0.00 -> 241.3 mm, vias 0 -> 2
- net col0: track 0.06 -> 203.8 mm
- net +5V: track 0.00 -> 180.6 mm, vias 0 -> 6
- net LED_1: track 0.00 -> 147.9 mm, vias 0 -> 2
- net LED_2: track 0.00 -> 140.8 mm, vias 0 -> 2
- net LED_3: track 0.00 -> 133.8 mm, vias 0 -> 2
- net row4: track 2.36 -> 124.3 mm, vias 0 -> 2
- net col5: track 3.59 -> 95.2 mm
- net RST: track 0.00 -> 86.0 mm, vias 0 -> 3
- net Net-(D_SPACE38-Pad2): track 70.4 -> 3.66 mm
- net col11: track 91.9 -> 151.4 mm
- net col10: track 72.6 -> 132.1 mm
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Other:
- board text removed: "1"
- board text removed: "1.5u"
- board text removed: "2"
- board text removed: "3"
