File: V4LPH4.kicad_sch (KiCad schematic)
At the start: 132 parts, among them SW1 SW_PUSH, SW2 SW_PUSH, U1 SRV05-4, U2 ATmega32U4-M, X1 Crystal_GND24_Small

Commit message: route
Parts:
- K_SPACE41, K_SPACE46: footprint MX_Only:MXOnly-1U-NoLED -> MX_Only:MXOnly-1.25U-NoLED
- K_SPACE42, K_SPACE45: footprint MX_Only:MXOnly-1.25U-NoLED -> MX_Only:MXOnly-1U-NoLED
- K_SPACE43: footprint MX_Only:MXOnly-1.75U-NoLED -> MX_Only:MXOnly-1.5U-NoLED
- K_SPACE44: footprint MX_Only:MXOnly-1.5U-NoLED -> MX_Only:MXOnly-1.75U-NoLED
Connections:
- net PD2 is gone; now on net row0: U2.20 (PD2)
- net LED_1: now also U2.9 (PB1)
- net LED_2: now also U2.10 (PB2)
- net LED_3: now also U2.11 (PB3)
- net col10: now also K_SPACE46.1; no longer K_SPACE47.1
- net col11: now also K_SPACE47.1; no longer K_SPACE33.1
- net col12: now also K_SPACE33.1
- net col5: now also U2.37 (PF6); no longer U2.8 (PB0)
- net col7: no longer K_SPACE44.1
- net col8: now also K_SPACE44.1; no longer K_SPACE45.1
- net col9: now also K_SPACE45.1; no longer K_SPACE46.1
- net row0: no longer U2.12 (PB7)
- net row1: now also U2.30 (PB6); no longer U2.37 (PF6)
- net row2: now also U2.31 (PC6); no longer U2.30 (PB6)
- net row3: now also U2.32 (PC7); no longer U2.31 (PC6)
- net row4: now also U2.12 (PB7); no longer U2.36 (PF7)
- net PD5: no longer names the net of U2.22 (PD5)
Other:
- moved on the sheet: D_SPACE20, D_SPACE44, D_SPACE45, D_SPACE46, D_SPACE47, K_SPACE33, K_SPACE44, K_SPACE45, K_SPACE46, K_SPACE47
